Commit message: fix(low_level,resources): 同步 v1.3.0 语音示例修复与 URDF 模型尺寸修正
- low_level 语音示例:
  - e7_voice_pub (Python/C++): 去掉硬编码音频路径 /root/test2.flac，
    改为从命令行参数接收文件路径
  - e8_voice_sub (Python): 补全 WAV 录制功能（此前只有声明未实现）
  - e8_voice_sub (C++): 修正注释中的示例编号 e9 -> e8，移除无用 include
- resources: 更新点足与轮足构型的 URDF/xacro 模型尺寸
  (hip_y 0.07 -> 0.062, 腿部偏移 0.08895 -> 0.097)

File: resources/dobot_quad/urdf/dobot_quad_ros.urdf (robot description, URDF)
Before this commit: robot dobot_quad, 17 links, 16 joints
Joints:
- joint joint_front_left_abad: origin xyz=0.2525 0.07 0 rpy=0 0 0 -> xyz=0.2525 0.062 0 rpy=0 0 0
- joint joint_front_left_thigh_pitch: origin xyz=0.0  0.08895 0.0 rpy=0 0 0 -> xyz=0.0  0.097 0.0 rpy=0 0 0
- joint joint_front_right_abad: origin xyz=0.2525 -0.07 0 rpy=0 0 0 -> xyz=0.2525 -0.062 0 rpy=0 0 0
- joint joint_front_right_thigh_pitch: origin xyz=0.0  -0.08895 0.0 rpy=0 0 0 -> xyz=0.0  -0.097 0.0 rpy=0 0 0
- joint joint_rear_left_abad: origin xyz=-0.2525 0.07 0 rpy=0 0 0 -> xyz=-0.2525 0.062 0 rpy=0 0 0
- joint joint_rear_left_thigh_pitch: origin xyz=-0.0  0.08895 0.0 rpy=0 0 0 -> xyz=-0.0  0.097 0.0 rpy=0 0 0
- joint joint_rear_right_abad: origin xyz=-0.2525 -0.07 0 rpy=0 0 0 -> xyz=-0.2525 -0.062 0 rpy=0 0 0
- joint joint_rear_right_thigh_pitch: origin xyz=-0.0  -0.08895 0.0 rpy=0 0 0 -> xyz=-0.0  -0.097 0.0 rpy=0 0 0

File: resources/dobot_quad/xacro/dobot_quad.xacro (robot description, xacro)
@@ -56,7 +56,7 @@
   </joint>
   <xacro:include filename="$(find dobot_quad)/xacro/leg_dobot_quad_collision_complete.xacro"/>
-  <xacro:leg_dobot_quad name="front_left"  hip_x="0.2525" hip_y="0.07"  x_sign="1" y_sign="1"/>
-  <xacro:leg_dobot_quad name="front_right" hip_x="0.2525" hip_y="-0.07" x_sign="1" y_sign="-1"/>
-  <xacro:leg_dobot_quad name="rear_left"  hip_x="-0.2525" hip_y="0.07" x_sign="-1" y_sign="1"/>
-  <xacro:leg_dobot_quad name="rear_right" hip_x="-0.2525" hip_y="-0.07" x_sign="-1" y_sign="-1"/>
+  <xacro:leg_dobot_quad name="front_left"  hip_x="0.2525" hip_y="0.062"  x_sign="1" y_sign="1"/>
+  <xacro:leg_dobot_quad name="front_right" hip_x="0.2525" hip_y="-0.062" x_sign="1" y_sign="-1"/>
+  <xacro:leg_dobot_quad name="rear_left"  hip_x="-0.2525" hip_y="0.062" x_sign="-1" y_sign="1"/>
+  <xacro:leg_dobot_quad name="rear_right" hip_x="-0.2525" hip_y="-0.062" x_sign="-1" y_sign="-1"/>
 </robot>

File: resources/dobot_quad/xacro/leg_dobot_quad_collision_complete.xacro (robot description, xacro)
@@ -108,5 +108,5 @@
  </link>
  <joint name="joint_${name}_thigh_pitch" type="revolute">
-   <origin xyz="${0.0*x_sign}  ${0.08895*y_sign} 0.0" rpy="0 0 0" />
+   <origin xyz="${0.0*x_sign}  ${0.097*y_sign} 0.0" rpy="0 0 0" />
    <parent
      link="link_${name}_hip" />

File: resources/dobot_quad_wheel/urdf/dobot_quad_wheel_ros.urdf (robot description, URDF)
Before this commit: robot dobot_quad_wheel, 17 links, 16 joints
Joints:
- joint joint_front_left_abad: origin xyz=0.2525 0.07 0 rpy=0 0 0 -> xyz=0.2525 0.062 0 rpy=0 0 0
- joint joint_front_left_thigh_pitch: origin xyz=0.0  0.08895 0.0 rpy=0 0 0 -> xyz=0.0  0.097 0.0 rpy=0 0 0
- joint joint_front_right_abad: origin xyz=0.2525 -0.07 0 rpy=0 0 0 -> xyz=0.2525 -0.062 0 rpy=0 0 0
- joint joint_front_right_thigh_pitch: origin xyz=0.0  -0.08895 0.0 rpy=0 0 0 -> xyz=0.0  -0.097 0.0 rpy=0 0 0
- joint joint_rear_left_abad: origin xyz=-0.2525 0.07 0 rpy=0 0 0 -> xyz=-0.2525 0.062 0 rpy=0 0 0
- joint joint_rear_left_thigh_pitch: origin xyz=-0.0  0.08895 0.0 rpy=0 0 0 -> xyz=-0.0  0.097 0.0 rpy=0 0 0
- joint joint_rear_right_abad: origin xyz=-0.2525 -0.07 0 rpy=0 0 0 -> xyz=-0.2525 -0.062 0 rpy=0 0 0
- joint joint_rear_right_thigh_pitch: origin xyz=-0.0  -0.08895 0.0 rpy=0 0 0 -> xyz=-0.0  -0.097 0.0 rpy=0 0 0

File: resources/dobot_quad_wheel/xacro/dobot_quad_wheel.xacro (robot description, xacro)
@@ -56,7 +56,7 @@
   </joint>
   <xacro:include filename="$(find dobot_quad_wheel)/xacro/leg_dobot_quad_collision_complete.xacro"/>
-  <xacro:leg_dobot_quad name="front_left"  hip_x="0.2525" hip_y="0.07"  x_sign="1" y_sign="1"/>
-  <xacro:leg_dobot_quad name="front_right" hip_x="0.2525" hip_y="-0.07" x_sign="1" y_sign="-1"/>
-  <xacro:leg_dobot_quad name="rear_left"  hip_x="-0.2525" hip_y="0.07" x_sign="-1" y_sign="1"/>
-  <xacro:leg_dobot_quad name="rear_right" hip_x="-0.2525" hip_y="-0.07" x_sign="-1" y_sign="-1"/>
+  <xacro:leg_dobot_quad name="front_left"  hip_x="0.2525" hip_y="0.062"  x_sign="1" y_sign="1"/>
+  <xacro:leg_dobot_quad name="front_right" hip_x="0.2525" hip_y="-0.062" x_sign="1" y_sign="-1"/>
+  <xacro:leg_dobot_quad name="rear_left"  hip_x="-0.2525" hip_y="0.062" x_sign="-1" y_sign="1"/>
+  <xacro:leg_dobot_quad name="rear_right" hip_x="-0.2525" hip_y="-0.062" x_sign="-1" y_sign="-1"/>
 </robot>

File: resources/dobot_quad_wheel/xacro/leg_dobot_quad_collision_complete.xacro (robot description, xacro)
@@ -108,5 +108,5 @@
  </link>
  <joint name="joint_${name}_thigh_pitch" type="revolute">
-   <origin xyz="${0.0*x_sign}  ${0.08895*y_sign} 0.0" rpy="0 0 0" />
+   <origin xyz="${0.0*x_sign}  ${0.097*y_sign} 0.0" rpy="0 0 0" />
    <parent
      link="link_${name}_hip" />
